File: pcb/final macropad.kicad_pcb (KiCad board)
At the start: 2 copper layers, 64.7 x 63.5 mm, 19 parts, among them J1 OLED Module, SW1 SW_Push, SW2 SW_Push, SW3 SW_Push, SW4 SW_Push, SW5 SW_Push, SW6 SW_Push, U1 Sparkfun_Pro_Micro

Commit message: finished up firmware
Parts:
- added R7: 1k, Resistor_THT:R_Axial_DIN0207_L6.3mm_D2.5mm_P7.62mm_Horizontal, B.Cu at (127.6, 73.8)
- added R8: 1k, Resistor_THT:R_Axial_DIN0207_L6.3mm_D2.5mm_P7.62mm_Horizontal, B.Cu at (127.6, 76.9)
- R1, R2, R3, R4: value 1k -> 4.7k
- R5, R6: value 1k -> 4.7
Routing:
- net SDA: track 46.8 -> 74.6 mm
- net SCL: track 43.2 -> 67.5 mm
- net +5V: track 190.7 -> 204.9 mm
- net Key 1: track 64.7 -> 66.4 mm

Commit message: added gerber files
Parts:
- removed the REF** at (175.6, 58.6)
- R5, R6: value 4.7 -> 4.7k
- moved G*** 0.76 mm to (165.4, 67.6)
Other:
- board text added: "5V"
- board text added: "GND"
- board text added: "SCL"
- board text added: "SDA"
- board text added: "SW1"
- board text added: "SW2"
- board text added: "SW3"
- board text added: "SW4"
- board text added: "SW5"
- board text added: "SW6"
Changed lines of the file:
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@@
 			(plot_on_all_layers_selection 0x00000000_00000000_00000000_00000000)
 			(disableapertmacros no)
-			(usegerberextensions no)
+			(usegerberextensions yes)
 			(usegerberattributes yes)
 			(usegerberadvancedattributes yes)
-			(creategerberjobfile yes)
+			(creategerberjobfile no)
 			(dashed_line_dash_ratio 12.000000)
 			(dashed_line_gap_ratio 3.000000)
@@
 			(outputformat 1)
 			(mirror no)
-			(drillshape 1)
+			(drillshape 0)
 			(scaleselection 1)
-			(outputdirectory "")
+			(outputdirectory "../Production/gerbers/")
 		)
 	)
@@
 		(property "Reference" "SW6"
 			(at 0 3.175 0)
-			(layer "B.Fab")
+			(layer "F.SilkS")
 			(effects
 				(font
@@
 					(thickness 0.15)
 				)
-				(justify mirror)
 			)
 		)
@@
 		(property "Reference" "SW3"
 			(at 0 3.175 0)
-			(layer "B.Fab")
+			(layer "F.SilkS")
 			(effects
 				(font
@@
 					(thickness 0.15)
 				)
-				(justify mirror)
 			)
 		)
@@
 		(property "Reference" "SW4"
 			(at 0 3.175 0)
-			(layer "B.Fab")
+			(layer "F.SilkS")
 			(effects
 				(font
@@
 					(thickness 0.15)
 				)
-				(justify mirror)
 			)
 		)
@@
 	(footprint "Silkscreen:zizhuo pcb"
 		(layer "F.Cu")
-		(at 164.6936 67.346207 90)
+		(at 165.395554 67.625607 90)
 		(property "Reference" "G***"
 			(at 0 0 90)
@@
 			(effects
 				(font
-					(size 1.5 1.5)
-					(thickness 0.3)
+					(size 1 1)
+					(thickness 0.15)
 				)
 			)
@@
 			(effects
 				(font
-					(size 1.5 1.5)
-					(thickness 0.3)
+					(size 1 1)
+					(thickness 0.15)
 				)
 			)
@@
 		(property "Reference" "SW1"
 			(at 0 3.175 0)
-			(layer "B.Fab")
+			(layer "F.SilkS")
 			(effects
 				(font
@@
 					(thickness 0.15)
 				)
-				(justify mirror)
 			)
 		)
@@
 		(property "Reference" "SW2"
 			(at 0 3.175 0)
-			(layer "B.Fab")
+			(layer "F.SilkS")
 			(effects
 				(font
@@
 					(thickness 0.15)
 				)
-				(justify mirror)
 			)
 		)
@@
 		(property "Reference" "SW5"
 			(at 0 3.175 0)
-			(layer "B.Fab")
+			(layer "F.SilkS")
 			(effects
 				(font
@@
 					(thickness 0.15)
 				)
-				(justify mirror)
 			)
 		)
@@
 		)
 	)
-	(footprint "MountingHole:MountingHole_2.2mm_M2_DIN965"
-		(layer "F.Cu")
-		(at 175.5648 58.6486)
-		(descr "Mounting Hole 2.2mm, M2, no annular, generated by kicad-footprint-generator mountinghole.py")
-		(tags "mountinghole M2 DIN965")
-		(property "Reference" "REF**"
-			(at 0 -2.85 0)
-			(layer "F.SilkS")
-			(hide yes)
-			(effects
-				(font
-					(size 1 1)
-					(thickness 0.15)
-				)
-			)
-		)
-		(property "Value" "MountingHole_2.2mm_M2_DIN965"
-			(at 0 2.85 0)
-			(layer "F.Fab")
-			(hide yes)
-			(effects
-				(font
-					(size 1 1)
-					(thickness 0.15)
-				)
-			)
-		)
-		(property "Datasheet" ""
-			(at 0 0 0)
-			(layer "F.Fab")
-			(hide yes)
-			(effects
-				(font
-					(size 1.27 1.27)
-					(thickness 0.15)
-				)
-			)
-		)
-		(property "Description" ""
-			(at 0 0 0)
-			(layer "F.Fab")
-			(hide yes)
-			(effects
-				(font
-					(size 1.27 1.27)
-					(thickness 0.15)
-				)
-			)
-		)
-		(attr exclude_from_pos_files exclude_from_bom)
-		(fp_circle
-			(center 0 0)
-			(end 2.15 0)
-			(stroke
-				(width 0.05)
-				(type solid)
-			)
-			(fill no)
-			(layer "F.CrtYd")
-		)
-		(pad "" np_thru_hole circle
-			(at 0 0)
-			(size 2.2 2.2)
-			(drill 2.2)
-			(layers "*.Cu" "*.Mask")
-		)
-		(embedded_fonts no)
-	)
 	(footprint "Arduino:Sparkfun_Pro_Micro"
 		(layer "B.Cu")
@@
 			(at 7.62 5.08 90)
 			(layer "B.SilkS")
+			(hide yes)
 			(effects
 				(font
@@
 		(property "Value" "1k"
 			(at 3.81 2.0828 0)
-			(layer "B.Fab")
+			(layer "B.SilkS")
 			(effects
 				(font
@@
 		(fp_text user "${REFERENCE}"
 			(at 3.81 0 0)
-			(layer "B.Fab")
+			(layer "B.SilkS")
 			(effects
 				(font
@@
 			)
 		)
-		(property "Value" "4.7"
+		(property "Value" "4.7k"
 			(at 3.81 -2.37 0)
-			(layer "B.Fab")
+			(layer "B.SilkS")
 			(effects
 				(font
@@
 		(property "Value" "4.7k"
 			(at 3.81 -2.37 0)
-			(layer "B.Fab")
+			(layer "B.SilkS")
 			(effects
 				(font
@@
 		(property "Value" "4.7k"
 			(at 3.81 -2.37 0)
-			(layer "B.Fab")
+			(layer "B.SilkS")
 			(effects
 				(font
@@
 			)
 		)
-		(property "Value" "4.7"
+		(property "Value" "4.7k"
 			(at 3.81 -2.37 0)
-			(layer "B.Fab")
+			(layer "B.SilkS")
 			(effects
 				(font
@@
 		(property "Value" "4.7k"
 			(at 3.81 -2.37 0)
-			(layer "B.Fab")
+			(layer "B.SilkS")
 			(effects
 				(font
@@
 		(property "Value" "4.7k"
 			(at 3.81 -2.37 0)
-			(layer "B.Fab")
+			(layer "B.SilkS")
 			(effects
 				(font
@@
 		(property "Value" "1k"
 			(at 3.81 -2.37 0)
-			(layer "B.Fab")
+			(layer "B.SilkS")
 			(effects
 				(font
@@
 		(fp_text user "${REFERENCE}"
 			(at 3.81 0 0)
-			(layer "B.Fab")
+			(layer "B.SilkS")
 			(effects
 				(font
@@
 		(layer "Edge.Cuts")
 	)
+	(gr_text "SCL"
+		(at 156.9466 76.8604 0)
+		(layer "F.SilkS")
+		(effects
+			(font
+				(size 1 1)
+				(thickness 0.15)
+			)
+			(justify left bottom)
+		)
+	)
 	(gr_text "Happy Birthday Zizhuo!\n25/03/2026"
-		(at 174.9298 66.5226 90)
+		(at 176.1998 66.294 90)
 		(layer "F.SilkS")
 		(effects
 			(font
-				(size 0.8 0.8)
-				(thickness 0.09375)
+				(size 1 1)
+				(thickness 0.15)
+				(bold yes)
 			)
 			(justify bottom)
 		)
 	)
+	(gr_text "SW5"
+		(at 141.5288 76.8604 0)
+		(layer "F.SilkS")
+		(effects
+			(font
+				(size 1 1)
+				(thickness 0.15)
+			)
+			(justify left bottom)
+		)
+	)
+	(gr_text "5V"
+		(at 116.7892 68.5038 90)
+		(layer "F.SilkS")
+		(effects
+			(font
+				(size 1 1)
+				(thickness 0.15)
+			)
+			(justify left bottom)
+		)
+	)
+	(gr_text "SW3"
+		(at 147.049067 61.6966 0)
+		(layer "F.SilkS")
+		(effects
+			(font
+				(size 1 1)
+				(thickness 0.15)
+			)
+			(justify left bottom)
+		)
+	)
+	(gr_text "SW4"
+		(at 144.5768 76.8604 0)
+		(layer "F.SilkS")
+		(effects
+			(font
+				(size 1 1)
+				(thickness 0.15)
+			)
+			(justify left bottom)
+		)
+	)
+	(gr_text "SW6"
+		(at 140.97 61.6966 0)
+		(layer "F.SilkS")
+		(effects
+			(font
+				(size 1 1)
+				(thickness 0.15)
+			)
+			(justify left bottom)
+		)
+	)
+	(gr_text "SDA"
+		(at 116.7892 63.881 90)
+		(layer "F.SilkS")
+		(effects
+			(font
+				(size 1 1)
+				(thickness 0.15)
+			)
+			(justify left bottom)
+		)
+	)
+	(gr_text "GND"
+		(at 116.7892 71.8058 90)
+		(layer "F.SilkS")
+		(effects
+			(font
+				(size 1 1)
+				(thickness 0.15)
+			)
+			(justify left bottom)
+		)
+	)
+	(gr_text "SDA"
+		(at 159.8168 76.8604 0)
+		(layer "F.SilkS")
+		(effects
+			(font
+				(size 1 1)
+				(thickness 0.15)
+			)
+			(justify left bottom)
+		)
+	)
+	(gr_text "SW2"
+		(at 144.009533 61.6966 0)
+		(layer "F.SilkS")
+		(effects
+			(font
+				(size 1 1)
+				(thickness 0.15)
+			)
+			(justify left bottom)
+		)
+	)
+	(gr_text "SCL"
+		(at 116.7892 66.6242 90)
+		(layer "F.SilkS")
+		(effects
+			(font
+				(size 1 1)
+				(thickness 0.15)
+			)
+			(justify left bottom)
+		)
+	)
+	(gr_text "SW1"
+		(at 150.0886 61.6966 0)
+		(layer "F.SilkS")
+		(effects
+			(font
+				(size 1 1)
+				(thickness 0.15)
+			)
+			(justify left bottom)
+		)
+	)
