File: pcb/final macropad.kicad_sch (KiCad schematic)
At the start: 14 parts, among them J1 OLED Module, SW1 SW_Push, SW2 SW_Push, SW3 SW_Push, SW4 SW_Push, SW5 SW_Push, SW6 SW_Push, U1 Sparkfun_Pro_Micro

Commit message: replaced footprints of switches, routed pcb
Parts:
- SW1, SW2, SW3, SW4, SW5, SW6: footprint Button_Switch_Keyboard:SW_Cherry_MX_1.00u_PCB -> MX_Only:MXOnly-1U-Hotswap
Changed lines of the file:
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@@
 			)
 		)
-		(property "Footprint" "Button_Switch_Keyboard:SW_Cherry_MX_1.00u_PCB"
+		(property "Footprint" "MX_Only:MXOnly-1U-Hotswap"
 			(at 223.52 125.73 0)
 			(effects
@@
 			)
 		)
-		(property "Footprint" "Button_Switch_Keyboard:SW_Cherry_MX_1.00u_PCB"
+		(property "Footprint" "MX_Only:MXOnly-1U-Hotswap"
 			(at 223.52 107.95 0)
 			(effects
@@
 			)
 		)
-		(property "Footprint" "Button_Switch_Keyboard:SW_Cherry_MX_1.00u_PCB"
+		(property "Footprint" "MX_Only:MXOnly-1U-Hotswap"
 			(at 223.52 116.84 0)
 			(effects
@@
 			)
 		)
-		(property "Footprint" "Button_Switch_Keyboard:SW_Cherry_MX_1.00u_PCB"
+		(property "Footprint" "MX_Only:MXOnly-1U-Hotswap"
 			(at 223.52 134.62 0)
 			(effects
@@
 			)
 		)
-		(property "Footprint" "Button_Switch_Keyboard:SW_Cherry_MX_1.00u_PCB"
+		(property "Footprint" "MX_Only:MXOnly-1U-Hotswap"
 			(at 223.52 99.06 0)
 			(effects
@@
 			)
 		)
-		(property "Footprint" "Button_Switch_Keyboard:SW_Cherry_MX_1.00u_PCB"
+		(property "Footprint" "MX_Only:MXOnly-1U-Hotswap"
 			(at 223.52 90.17 0)
 			(effects

Commit message: finished up firmware
Parts:
- added R7, R8: 1k, Resistor_THT:R_Axial_DIN0207_L6.3mm_D2.5mm_P7.62mm_Horizontal, symbol Device:R
- R1, R2, R3, R4: value 1k -> 4.7k
- R5, R6: value 1k -> 4.7
Connections:
- net +5V: now also R7.1, R8.1
- net SCL: now also R7.2
- net SDA: now also R8.2

Commit message: updated drawing sheet
Other:
- company: (none) -> Ng Yu Heng, Hong Guo Feng
- title: (none) -> Zizhuo Macropad
Changed lines of the file:
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@@
 	(generator_version "9.0")
 	(paper "A4")
+	(title_block
+		(title "Zizhuo Macropad")
+		(date "2026-04-11")
+		(rev "2.2")
+		(company "Ng Yu Heng, Hong Guo Feng")
+		(comment 1 "Macropad Designed for Zizhuo's Birthday")
+	)
 	(rectangle
 		(start 140.97 72.39)
@@
 	)
 	(embedded_fonts no)
+	(embedded_files
+		(file
+			(name "zizhuopad.kicad_wks")
+			(type worksheet)
+			(data |KLUv/WABCW0UAPadXiEAtxsWHGS5ac4JWlhdTS3ZQeABQKzGkOeo5yaqqm4BIAJUAE0AWAB5xP/4
+				I/F/PDZP2td6sjdyvuOi4aLW7M+HluTXiobLou0nW37JvwAABASk6L2cVlZxKhs6RySrzvi97Nc9
+				BoxSiqiz9sW2zD4qAAKCMkTihB5oQ4VdYrKiVX/J//trIq7a8zKVMnhtv+ek98x+MwZf7NmzCoFY
+				/NrFt9/++Q6vCGevq/7r44jBWbt2eL3WOa2rdoZlVjZpf/a+rKr20bsPephQxF8nKqfZLiO/YFjV
+				EWolOpuUUuEwl03DcWgNLoIiXNZlXT0pzSxFL7DU1mkOzpbBYDgUoRn+niPnbMr+18E2deyXItBV
+				m2qmevX8vm9SRAHwF3doXzUBgaEqapZNBO0o28R0PXLEjVk3FM0yqTQWkE6zdNsGwWAYwkpMNMom
+				4R72AVrRe9uG2nVhTbpJOq4T33aVVhrafvcPZnBIDUKu6vfGjDudnfQsl82iWfxkA3Sg0UCHHJoS
+				UZAkSTpgRKTmqh58ydw6HOT34t+rqOyMQT7ZMIZ5T++YII8GygjjWC475yaGfEy0wcezeezaPDte
+				FmTpYs1iemriCcKR29dmmvPiTxPwqZzsKZRQk1nMhgj2ISCU8e7YIj9grRzOyKAhTJ76YcJiN8YV
+				Di6ZsjQail5KUUyWjVMH8QH3f6YWHNtMH72HdRikI6b+qClK05DLxnIf4RpAb23FYUFAe5j+RoUi
+				745wgN+e77VsIew8s3ALXfTKD8T2dXj0CQLPVJEgFXgLYS4AhghypzcfHgLGbhJovPoY+IwKAOo9
+				SNJU4UFKmxPyW5HATuaKYZsGjXri1qz1/zg+gn7y0QF/DEwV|
+			)
+			(checksum "FE3E7361A44BD2D0931D02A779DA6436")
+		)
+	)
 )
